Commit message: .

File: ros/src/cyton_description/urdf/cyton_gamma_1500_robot.xacro (robot description, xacro)
@@ -363,15 +363,11 @@
        rigidly to virtual_endeffector, representing the physical hydrophone
        probe used to measure ultrasound propagation at points on a skull
-       phantom. Visual/collision attachment only, by explicit user choice -
-       MoveIt's planning group tip_link deliberately stays at
-       virtual_endeffector (not the rod tip), so IK/Cartesian targets still
-       refer to the original wrist-mounted point; the rod's length (10cm)
-       must be accounted for manually when picking targets. Dimensions
-       below are nominal design values (10cm length, 4mm diameter), not
-       independently calibrated - verify against the physical probe if
-       precise real-world accuracy at the rod tip matters. Extends along
-       +Z, matching this URDF's existing convention (every joint's origin
-       in this chain has its dominant offset along the parent's +Z, i.e.
-       +Z is "outward along the arm's reach" throughout). -->
+       phantom. Dimensions are nominal design values (10cm length, 4mm
+       diameter), not independently calibrated - verify against the
+       physical probe if precise real-world accuracy at the rod tip
+       matters. Extends along +Z, matching this URDF's existing convention
+       (every joint's origin in this chain has its dominant offset along
+       the parent's +Z, i.e. +Z is "outward along the arm's reach"
+       throughout). -->
   <joint name="hydrophone_rod_joint" type="fixed">
     <parent link="virtual_endeffector"/>
@@ -396,3 +392,23 @@
     </collision>
   </link>
+  <!-- Rod-tip reference frame (2026-08-24): a zero-size frame at the FAR
+       end of the rod (z=0.10 relative to virtual_endeffector, matching
+       the cylinder's own far face). MoveIt's planning group tip_link now
+       points HERE (see cyton_gamma_1500.srdf), not virtual_endeffector -
+       reversing the original 2026-08-11 decision. IK/Cartesian targets
+       now refer to the actual physical probe tip directly; no more manual
+       10cm accounting when picking targets. This also fixes a real,
+       observed problem with the old setup: standoff was being measured
+       from virtual_endeffector, so the rod (extending 10cm further)
+       could be driven straight through a target surface even though the
+       commanded pose was nominally "10mm short" of it - the arm was
+       satisfying the standoff at the wrong point on itself. Now that the
+       tip itself is what's commanded to stop short, the rod naturally
+       clears the surface it's approaching. -->
+  <joint name="hydrophone_tip_joint" type="fixed">
+    <parent link="hydrophone_rod"/>
+    <child link="hydrophone_tip"/>
+    <origin rpy="0 0 0" xyz="0 0 0.10"/>
+  </joint>
+  <link name="hydrophone_tip"/>
 </robot>

File: ros/src/cyton_description/urdf/cyton_gamma_1500_robot_sim7dof.xacro (robot description, xacro)
@@ -1,37 +1,34 @@
-<?xml version="1.0" ?>
-<robot name="cyton_gamma_1500">
-  <!--
-    KINEMATIC CALIBRATION USED FOR STANDALONE IK
-    Updated 2026-08-06 with the fitted corrections from this project's NDI-
-    based kinematic calibration (see CLAUDE.md's kinematic-calibration
-    section for the full history/methodology). Per-joint <axis> and (for
-    elbow_pitch/shoulder_yaw/wrist_pitch) <origin xyz> below now reflect
-    those corrections; see each joint's own inline comment for the specific
-    change and its original nominal value.
-    URDF joint              Motor ID   zero tick   safe ticks     scale     corrected?
-    shoulder_roll_joint        0          2048      276..3772   0.988203   tilt only (offset skipped: base-frame degeneracy)
-    shoulder_pitch_joint       1          2047      851..3231   1.001931   offset+scale+tilt
-    shoulder_yaw_joint         2          2060      912..3327   0.964711   offset+scale+tilt+origin
-    elbow_pitch_joint          3          2102      799..3307   1.014467   offset+scale+tilt+origin (widened 2026-08-07, was 829..3277, see joint's own comment)
-    elbow_yaw_joint             4          2078     2060..2130  1.0        NONE — deliberately locked near
-                                                                              midpoint in production; its own fit
-                                                                              is poorly identified (joint barely
-                                                                              moved in the dataset used to fit it)
-    wrist_pitch_joint          5          2042      751..3344   1.006796   offset+scale+tilt+origin
-    wrist_roll_joint           6          2048      335..3761   1.002933   tilt only (offset skipped: tool-frame degeneracy)
-    Motor ID 7 is the gripper and is intentionally excluded from the
-    base_link -> virtual_endeffector IK chain.
-    NOT integrated here, and not representable in a static URDF at all:
-    joint-coupling (3 terms), gravity/elastostatic deflection (7 terms), and
-    the shoulder_pitch Fourier term — all pose-dependent, would need a
-    real-time correction layer in whatever control stack ends up driving
-    this robot, not a geometry change. Backlash compensation is separately
-    already implemented as C++ logic in src/dynamixel_motor.cpp (per-joint
-    overshoot on direction reversal) and needs porting into that same
-    control layer, not this file.
-    The limits below were converted using 4096 ticks per revolution.
-    Joint axes and positive directions must still be verified physically.
-    velocity=1.0 is retained as an unverified planning placeholder.
-  -->
+<?xml version="1.0"?>
+<!--
+  SIMULATION-ONLY 7-DOF variant (2026-08-24). Identical to the real,
+  deployed cyton_gamma_1500_robot.xacro (see that file's own header for
+  everything else - geometry provenance, what's not included, etc.)
+  except for ONE change: elbow_yaw_joint's <limit> is widened back to the
+  full original mechanical range (lower="-1.727262" upper="1.790156",
+  preserved in cyton_gamma_1500_robot.xacro's own elbow_yaw_joint comment)
+  instead of the ~4-degree production lock.
+  WHY THIS IS SAFE ONLY IN SIMULATION: elbow_yaw is locked in production
+  because that joint's own calibration fit was poorly identified (it
+  barely moved in the dataset used to fit it) - not because the joint
+  itself is mechanically unsafe to move. On hardware_type=mock_components,
+  ros2_control uses its own built-in mock_components/GenericSystem plugin
+  (see cyton_gamma_1500.ros2_control.xacro), which never invokes
+  cyton_hardware/CytonSystemHardware or robot_calibration.cpp's hardware-
+  level safety clamp at all - on mock, this URDF's <limit> tags are the
+  ONLY thing constraining joint range, so widening it here only affects
+  simulated/planned motion, never a real servo.
+  DO NOT combine this variant with hardware_type=real. Nothing in this
+  file enforces that by itself (a URDF fragment can't see the hardware_type
+  arg) - the launch-level guard is in cyton_moveit_config/launch/
+  demo.launch.py, which rejects urdf_variant=sim_7dof + hardware_type=real
+  outright. If you're adding a new way to launch this variant, add the
+  same guard there too.
+  DO NOT hand-edit any calibration number other than elbow_yaw_joint's
+  <limit> here - for everything else this must stay a straight copy of
+  cyton_gamma_1500_robot.xacro (and by extension,
+  references/cyton_gamma_1500_trac_ik.urdf); keep both in sync by hand
+  if either's non-elbow_yaw calibration ever changes.
+-->
+<robot name="cyton_gamma_1500" xmlns:xacro="http://www.ros.org/wiki/xacro">
   <!-- base -->
   <link name="base_footprint">
@@ -55,5 +52,5 @@
       <origin rpy="0 0 0" xyz="0 0 0"/>
       <geometry>
-        <mesh filename="package://cyton_gamma_1500_description/meshes/base.dae"/>
+        <mesh filename="package://cyton_description/meshes/base.dae"/>
       </geometry>
     </visual>
@@ -86,10 +83,8 @@
       upper="2.644583"
       velocity="1.0"/>
-    <!-- Axis tilt correction applied 2026-08-06, from the kinematic
-         calibration fit (see CLAUDE.md's kinematic-calibration section).
-         Original nominal axis: 0 0 1. (This joint's fitted zero-offset was
-         NOT applied to zeroTick in robot_calibration.cpp — entangled with
-         the calibration-time base frame's rotation — but axis tilt does
-         not share that degeneracy and is safe to apply here.) -->
+    <!-- Axis tilt correction (2026-08-06 kinematic calibration fit).
+         Original nominal axis: 0 0 1. Fitted zero-offset NOT applied
+         (base-frame degeneracy)  -  axis tilt does not share that
+         degeneracy and is safe to apply here. -->
     <axis xyz="0.013792 0.014877 0.999794"/>
   </joint>
@@ -98,5 +93,5 @@
       <origin rpy="1.5708 0 0.384" xyz="0 0 0"/>
       <geometry>
-        <mesh filename="package://cyton_gamma_1500_description/meshes/shoulder_roll.dae"/>
+        <mesh filename="package://cyton_description/meshes/shoulder_roll.dae"/>
       </geometry>
     </visual>
@@ -123,6 +118,5 @@
       upper="1.814699"
       velocity="1.0"/>
-    <!-- Axis tilt correction applied 2026-08-06, from the kinematic
-         calibration fit (see CLAUDE.md's kinematic-calibration section).
+    <!-- Axis tilt correction (2026-08-06 kinematic calibration fit).
          Original nominal axis: 1 0 0. -->
     <axis xyz="0.998997 -0.043573 -0.010357"/>
@@ -132,5 +126,5 @@
       <origin rpy="1.5708 0 0" xyz="0 0 0"/>
       <geometry>
-        <mesh filename="package://cyton_gamma_1500_description/meshes/shoulder_pitch.dae"/>
+        <mesh filename="package://cyton_description/meshes/shoulder_pitch.dae"/>
       </geometry>
     </visual>
@@ -151,8 +145,7 @@
     <parent link="shoulder_pitch"/>
     <child link="shoulder_yaw"/>
-    <!-- Origin and axis tilt corrections applied 2026-08-06, from the
-         kinematic calibration fit (see CLAUDE.md's kinematic-calibration
-         section). Original nominal origin xyz: -0.0215 -0.0205 0.1255
-         (only x,z corrected; y untouched by the fit's parameterization).
+    <!-- Origin and axis tilt corrections (2026-08-06 kinematic calibration
+         fit). Original nominal origin xyz: -0.0215 -0.0205 0.1255 (only
+         x,z corrected; y untouched by the fit's parameterization).
          Original nominal axis: 0 -1 0. -->
     <origin rpy="0 0 0" xyz="-0.02478414 -0.0205 0.1308452"/>
@@ -168,5 +161,5 @@
       <origin rpy="1.5708 0 -1.5708" xyz="0 0 0.0"/>
       <geometry>
-        <mesh filename="package://cyton_gamma_1500_description/meshes/shoulder_yaw.dae"/>
+        <mesh filename="package://cyton_description/meshes/shoulder_yaw.dae"/>
       </geometry>
     </visual>
@@ -187,24 +180,18 @@
     <parent link="shoulder_yaw"/>
     <child link="elbow_pitch"/>
-    <!-- Origin and axis tilt corrections applied 2026-08-06, from the
-         kinematic calibration fit (see CLAUDE.md's kinematic-calibration
-         section). Original nominal origin xyz: 0.018 0.0206 0.1158.
+    <!-- Origin and axis tilt corrections (2026-08-06 kinematic calibration
+         fit). Original nominal origin xyz: 0.018 0.0206 0.1158.
          Original nominal axis: 1 0 0. -->
     <origin rpy="0 0 0" xyz="0.01656849 0.02722018 0.11356304"/>
     <!-- Limit widened 2026-08-07 (was lower="-1.961961" upper="1.788622")
          to add a 30-tick margin on each side of jointCalibrations[3]'s
-         minTick/maxTick (robot_calibration.cpp) - real-hardware MoveIt
+         minTick/maxTick (robot_calibration.cpp)  -  real-hardware MoveIt
          sessions repeatedly showed the arm's actual settled position
          landing a few ticks up to ~25 ticks past the exact hand-verified
-         extreme (ordinary servo settling/backlash noise), which
-         MoveIt's CheckStartStateBounds check has zero tolerance for and
-         will not plan past. Recomputed directly from the widened
-         [799, 3307] tick range, not just delta-adjusted from the old
-         values - doing so surfaced that the *previous* limit here had
-         quietly drifted ~12-26 ticks tighter than jointCalibrations'
-         then-current [829, 3277] anyway (likely stale from an earlier
-         zeroTick/scale revision that was never propagated here), so this
-         edit also fixes that pre-existing mismatch, not just adds
-         margin. -->
+         extreme (ordinary servo settling/backlash noise), which MoveIt's
+         CheckStartStateBounds check has zero tolerance for. See
+         references/cyton_gamma_1500_trac_ik.urdf's matching joint comment
+         for the full explanation, including a pre-existing (now fixed)
+         mismatch this recomputation also caught. -->
     <limit
       effort="100.0"
@@ -218,5 +205,5 @@
       <origin rpy="1.5708 0 3.1416" xyz="0 0 0"/>
       <geometry>
-        <mesh filename="package://cyton_gamma_1500_description/meshes/elbow_pitch.dae"/>
+        <mesh filename="package://cyton_description/meshes/elbow_pitch.dae"/>
       </geometry>
     </visual>
@@ -237,28 +224,20 @@
     <parent link="elbow_pitch"/>
     <child link="elbow_yaw"/>
-    <!-- elbow_yaw_joint deliberately left UNCORRECTED (2026-08-06): this
-         joint is locked near its calibrated midpoint in production (see
-         src/robot_calibration.cpp's jointCalibrations comment and CLAUDE.md's
-         kinematic-calibration section, "reduced-DOF breakthrough") and barely
-         moved in the dataset used to fit it, so its own tilt/scale/offset
-         correction is poorly identified and not trustworthy — moot anyway
-         since it's not meant to move in real use. -->
+    <!-- elbow_yaw_joint's tilt/scale/offset correction is still left
+         UNCORRECTED here (same reasoning as the real calibrated file:
+         poorly identified, barely moved in the fit dataset) - only the
+         <limit> below differs from that file, per this file's own header
+         comment. -->
     <origin rpy="0 0 0" xyz="-0.0171 -0.018 0.09746"/>
-    <!-- Limit tightened 2026-08-06 to match this joint's hardware lock
-         (jointCalibrations[4]'s minTick/maxTick, robot_calibration.cpp)
-         — MUST stay consistent with that C++ range, not the original wide
-         mechanical limit, or MoveIt will plan trajectories the hardware
-         safety clamp will reject. Original wide limit was
-         lower="-1.727262" upper="1.790156".
-         Widened slightly again 2026-08-07 (was lower="-0.004602"
-         upper="0.056757") - 15 ticks of margin added each side of
-         jointCalibrations[4]'s range (now [2060, 2130]), same real-
-         hardware-settling-noise reasoning as elbow_pitch_joint's limit
-         above. Still a deliberately tiny ~4 degree window; this joint
-         stays "locked" in every practical sense. -->
-    <limit
-      effort="100.0"
-      lower="-0.027612"
-      upper="0.079767"
+    <!-- SIM-ONLY WIDENING (2026-08-24): full original mechanical range,
+         not the production hardware lock - see this file's own header
+         comment for why that's safe here (mock_components only) and
+         nowhere else. The production-locked value (for reference, and
+         what every OTHER urdf_variant still uses) is
+         lower="-0.027612" upper="0.079767". -->
+    <limit
+      effort="100.0"
+      lower="-1.727262"
+      upper="1.790156"
       velocity="1.0"/>
     <axis xyz="0 -1 0"/>
@@ -268,5 +247,5 @@
       <origin rpy="1.5708 0 1.5708" xyz="0 0 0"/>
       <geometry>
-        <mesh filename="package://cyton_gamma_1500_description/meshes/elbow_yaw.dae"/>
+        <mesh filename="package://cyton_description/meshes/elbow_yaw.dae"/>
       </geometry>
     </visual>
@@ -287,7 +266,6 @@
     <parent link="elbow_yaw"/>
     <child link="wrist_pitch"/>
-    <!-- Origin and axis tilt corrections applied 2026-08-06, from the
-         kinematic calibration fit (see CLAUDE.md's kinematic-calibration
-         section). Original nominal origin xyz: 0.02626 0.018 0.0718.
+    <!-- Origin and axis tilt corrections (2026-08-06 kinematic calibration
+         fit). Original nominal origin xyz: 0.02626 0.018 0.0718.
          Original nominal axis: 1 0 0. -->
     <origin rpy="0 0 0" xyz="0.02765348 0.01273746 0.07244612"/>
@@ -303,5 +281,5 @@
       <origin rpy="1.5708 0 1.5708" xyz="0 0 0"/>
       <geometry>
-        <mesh filename="package://cyton_gamma_1500_description/meshes/wrist_pitch.dae"/>
+        <mesh filename="package://cyton_description/meshes/wrist_pitch.dae"/>
       </geometry>
     </visual>
@@ -328,10 +306,8 @@
       upper="2.618505"
       velocity="1.0"/>
-    <!-- Axis tilt correction applied 2026-08-06, from the kinematic
-         calibration fit (see CLAUDE.md's kinematic-calibration section).
-         Original nominal axis: 0 0 1. (This joint's fitted zero-offset was
-         NOT applied to zeroTick in robot_calibration.cpp — entangled with
-         the calibration-time tool frame's rotation — but axis tilt does
-         not share that degeneracy and is safe to apply here.) -->
+    <!-- Axis tilt correction (2026-08-06 kinematic calibration fit).
+         Original nominal axis: 0 0 1. Fitted zero-offset NOT applied
+         (tool-frame degeneracy)  -  axis tilt does not share that
+         degeneracy and is safe to apply here. -->
     <axis xyz="-0.006451 -0.018572 0.999807"/>
   </joint>
@@ -340,5 +316,5 @@
       <origin rpy="3.1416 0 -1.5708" xyz="0 0 0"/>
       <geometry>
-        <mesh filename="package://cyton_gamma_1500_description/meshes/wrist_roll.dae"/>
+        <mesh filename="package://cyton_description/meshes/wrist_roll.dae"/>
       </geometry>
     </visual>

File: ros/src/cyton_description/urdf/cyton_gamma_1500_robot_uncalibrated.xacro (robot description, xacro)
@@ -377,15 +377,11 @@
        rigidly to virtual_endeffector, representing the physical hydrophone
        probe used to measure ultrasound propagation at points on a skull
-       phantom. Visual/collision attachment only, by explicit user choice -
-       MoveIt's planning group tip_link deliberately stays at
-       virtual_endeffector (not the rod tip), so IK/Cartesian targets still
-       refer to the original wrist-mounted point; the rod's length (10cm)
-       must be accounted for manually when picking targets. Dimensions
-       below are nominal design values (10cm length, 4mm diameter), not
-       independently calibrated - verify against the physical probe if
-       precise real-world accuracy at the rod tip matters. Extends along
-       +Z, matching this URDF's existing convention (every joint's origin
-       in this chain has its dominant offset along the parent's +Z, i.e.
-       +Z is "outward along the arm's reach" throughout). -->
+       phantom. Dimensions are nominal design values (10cm length, 4mm
+       diameter), not independently calibrated - verify against the
+       physical probe if precise real-world accuracy at the rod tip
+       matters. Extends along +Z, matching this URDF's existing convention
+       (every joint's origin in this chain has its dominant offset along
+       the parent's +Z, i.e. +Z is "outward along the arm's reach"
+       throughout). -->
   <joint name="hydrophone_rod_joint" type="fixed">
     <parent link="virtual_endeffector"/>
@@ -410,3 +406,16 @@
     </collision>
   </link>
+  <!-- Rod-tip reference frame (2026-08-24): a zero-size frame at the FAR
+       end of the rod (z=0.10 relative to virtual_endeffector, matching
+       the cylinder's own far face). MoveIt's planning group tip_link now
+       points HERE (see cyton_gamma_1500.srdf), not virtual_endeffector -
+       reversing the original 2026-08-11 decision. IK/Cartesian targets
+       now refer to the actual physical probe tip directly; no more manual
+       10cm accounting when picking targets. -->
+  <joint name="hydrophone_tip_joint" type="fixed">
+    <parent link="hydrophone_rod"/>
+    <child link="hydrophone_tip"/>
+    <origin rpy="0 0 0" xyz="0 0 0.10"/>
+  </joint>
+  <link name="hydrophone_tip"/>
 </robot>
