Commit message: fixed motor 5, which was the issue of offset

File: references/cyton_gamma_1500_trac_ik.urdf (robot description, URDF)
Before this commit: robot cyton_gamma_1500, 10 links, 9 joints
Joints:
- joint elbow_pitch_joint: limit lower=-1.833107 upper=1.833107 effort=100.0 velocity=1.0 -> lower=-1.961961 upper=1.788622 effort=100.0 velocity=1.0
- joint elbow_yaw_joint: limit lower=-1.833107 upper=1.833107 effort=100.0 velocity=1.0 -> lower=-1.727262 upper=1.790156 effort=100.0 velocity=1.0
- joint shoulder_pitch_joint: limit lower=-1.833107 upper=1.833107 effort=100.0 velocity=1.0 -> lower=-1.833107 upper=1.814699 effort=100.0 velocity=1.0
- joint shoulder_roll_joint: limit lower=-2.618505 upper=2.618505 effort=100.0 velocity=1.0 -> lower=-2.564816 upper=2.644583 effort=100.0 velocity=1.0
- joint shoulder_yaw_joint: limit lower=-1.846913 upper=1.846913 effort=100.0 velocity=1.0 -> lower=-1.770214 upper=1.934350 effort=100.0 velocity=1.0
- joint wrist_pitch_joint: limit lower=-1.833107 upper=1.833107 effort=100.0 velocity=1.0 -> lower=-1.989573 upper=1.988039 effort=100.0 velocity=1.0
- joint wrist_roll_joint: limit lower=-2.618505 upper=2.618505 effort=100.0 velocity=1.0 -> lower=-2.627709 upper=2.618505 effort=100.0 velocity=1.0

Commit message: urdf prepped for moveit

File: references/cyton_gamma_1500_trac_ik.urdf (robot description, URDF)
Before this commit: robot cyton_gamma_1500, 10 links, 9 joints
Joints:
- joint elbow_pitch_joint: axis 1 0 0 -> 0.999677 -0.024005 0.008304; origin xyz=0.018 0.0206 0.1158 rpy=0 0 0 -> xyz=0.01656849 0.02722018 0.11356304 rpy=0 0 0
- joint elbow_yaw_joint: limit lower=-1.727262 upper=1.790156 effort=100.0 velocity=1.0 -> lower=-0.004602 upper=0.056757 effort=100.0 velocity=1.0
- joint shoulder_pitch_joint: axis 1 0 0 -> 0.998997 -0.043573 -0.010357
- joint shoulder_roll_joint: axis 0 0 1 -> 0.013792 0.014877 0.999794
- joint shoulder_yaw_joint: axis 0 -1 0 -> -0.027678 -0.999437 0.018973; origin xyz=-0.0215 -0.0205 0.1255 rpy=0 0 0 -> xyz=-0.02478414 -0.0205 0.1308452 rpy=0 0 0
- joint wrist_pitch_joint: axis 1 0 0 -> 0.999044 0.042957 0.008105; origin xyz=0.02626 0.018 0.0718 rpy=0 0 0 -> xyz=0.02765348 0.01273746 0.07244612 rpy=0 0 0
- joint wrist_roll_joint: axis 0 0 1 -> -0.006451 -0.018572 0.999807

Commit message: more testing

File: references/cyton_gamma_1500_trac_ik.urdf (robot description, URDF)
Before this commit: robot cyton_gamma_1500, 10 links, 9 joints
Joints:
- joint elbow_pitch_joint: limit lower=-1.961961 upper=1.788622 effort=100.0 velocity=1.0 -> lower=-2.027693 upper=1.875188 effort=100.0 velocity=1.0
- joint elbow_yaw_joint: limit lower=-0.004602 upper=0.056757 effort=100.0 velocity=1.0 -> lower=-0.027612 upper=0.079767 effort=100.0 velocity=1.0

File: ros/src/cyton_description/urdf/cyton_gamma_1500_robot.xacro (robot description, xacro)
@@ -187,8 +187,18 @@
          Original nominal axis: 1 0 0. -->
     <origin rpy="0 0 0" xyz="0.01656849 0.02722018 0.11356304"/>
-    <limit
-      effort="100.0"
-      lower="-1.961961"
-      upper="1.788622"
+    <!-- Limit widened 2026-08-07 (was lower="-1.961961" upper="1.788622")
+         to add a 30-tick margin on each side of jointCalibrations[3]'s
+         minTick/maxTick (robot_calibration.cpp)  -  real-hardware MoveIt
+         sessions repeatedly showed the arm's actual settled position
+         landing a few ticks up to ~25 ticks past the exact hand-verified
+         extreme (ordinary servo settling/backlash noise), which MoveIt's
+         CheckStartStateBounds check has zero tolerance for. See
+         references/cyton_gamma_1500_trac_ik.urdf's matching joint comment
+         for the full explanation, including a pre-existing (now fixed)
+         mismatch this recomputation also caught. -->
+    <limit
+      effort="100.0"
+      lower="-2.027693"
+      upper="1.875188"
       velocity="1.0"/>
     <axis xyz="0.999677 -0.024005 0.008304"/>
@@ -227,13 +237,19 @@
     <origin rpy="0 0 0" xyz="-0.0171 -0.018 0.09746"/>
     <!-- Limit tightened 2026-08-06 to match this joint's hardware lock
-         (jointCalibrations[4]'s minTick/maxTick = 2075/2115 in
-         robot_calibration.cpp)  -  MUST stay consistent with that C++
-         range, not the original wide mechanical limit, or MoveIt will
-         plan trajectories the hardware safety clamp will reject. Original
-         wide limit was lower="-1.727262" upper="1.790156". -->
-    <limit
-      effort="100.0"
-      lower="-0.004602"
-      upper="0.056757"
+         (jointCalibrations[4]'s minTick/maxTick, robot_calibration.cpp)
+          -  MUST stay consistent with that C++ range, not the original
+         wide mechanical limit, or MoveIt will plan trajectories the
+         hardware safety clamp will reject. Original wide limit was
+         lower="-1.727262" upper="1.790156".
+         Widened slightly again 2026-08-07 (was lower="-0.004602"
+         upper="0.056757")  -  15 ticks of margin added each side of
+         jointCalibrations[4]'s range (now [2060, 2130]), same real-
+         hardware-settling-noise reasoning as elbow_pitch_joint's limit
+         above. Still a deliberately tiny ~4 degree window; this joint
+         stays "locked" in every practical sense. -->
+    <limit
+      effort="100.0"
+      lower="-0.027612"
+      upper="0.079767"
       velocity="1.0"/>
     <axis xyz="0 -1 0"/>

Commit message: easy points

File: references/cyton_gamma_1500_trac_ik.urdf (robot description, URDF)
Before this commit: robot cyton_gamma_1500, 10 links, 9 joints
Links:
- added link hydrophone_rod; collision cylinder length=0.10 radius=0.002; visual cylinder length=0.10 radius=0.002
Joints:
- added joint hydrophone_rod_joint: type fixed, parent virtual_endeffector, child hydrophone_rod, origin xyz=0 0 0 rpy=0 0 0

File: ros/src/cyton_description/urdf/cyton_gamma_1500_robot.xacro (robot description, xacro)
@@ -360,3 +360,39 @@
     </visual>
   </link>
+  <!-- Hydrophone probe rod (2026-08-11): a thin cylindrical rod attached
+       rigidly to virtual_endeffector, representing the physical hydrophone
+       probe used to measure ultrasound propagation at points on a skull
+       phantom. Visual/collision attachment only, by explicit user choice -
+       MoveIt's planning group tip_link deliberately stays at
+       virtual_endeffector (not the rod tip), so IK/Cartesian targets still
+       refer to the original wrist-mounted point; the rod's length (10cm)
+       must be accounted for manually when picking targets. Dimensions
+       below are nominal design values (10cm length, 4mm diameter), not
+       independently calibrated - verify against the physical probe if
+       precise real-world accuracy at the rod tip matters. Extends along
+       +Z, matching this URDF's existing convention (every joint's origin
+       in this chain has its dominant offset along the parent's +Z, i.e.
+       +Z is "outward along the arm's reach" throughout). -->
+  <joint name="hydrophone_rod_joint" type="fixed">
+    <parent link="virtual_endeffector"/>
+    <child link="hydrophone_rod"/>
+    <origin rpy="0 0 0" xyz="0 0 0"/>
+  </joint>
+  <link name="hydrophone_rod">
+    <visual>
+      <origin rpy="0 0 0" xyz="0 0 0.05"/>
+      <geometry>
+        <cylinder radius="0.002" length="0.10"/>
+      </geometry>
+      <material name="grey">
+        <color rgba="0.6 0.6 0.6 1.0"/>
+      </material>
+    </visual>
+    <collision>
+      <origin rpy="0 0 0" xyz="0 0 0.05"/>
+      <geometry>
+        <cylinder radius="0.002" length="0.10"/>
+      </geometry>
+    </collision>
+  </link>
 </robot>

Commit message: .

File: references/cyton_gamma_1500_trac_ik.urdf (robot description, URDF)
Before this commit: robot cyton_gamma_1500, 12 links, 11 joints
Links:
- link hydrophone_rod: geometry collision cylinder length=0.15 radius=0.002; visual cylinder length=0.15 radius=0.002
Joints:
- joint hydrophone_tip_joint: origin xyz=0 0 0.10 rpy=0 0 0 -> xyz=0 0 0.15 rpy=0 0 0

File: ros/src/cyton_description/urdf/cyton_gamma_1500_robot.xacro (robot description, xacro)
@@ -363,6 +363,9 @@
        rigidly to virtual_endeffector, representing the physical hydrophone
        probe used to measure ultrasound propagation at points on a skull
-       phantom. Dimensions are nominal design values (10cm length, 4mm
-       diameter), not independently calibrated - verify against the
+       phantom. Dimensions are nominal design values (15cm length, 4mm
+       diameter - lengthened from the original 10cm on 2026-08-25 to give
+       more standoff/collision clearance against the skull mesh, paired
+       with moving the skull's registration 10cm farther from base_link),
+       not independently calibrated - verify against the
        physical probe if precise real-world accuracy at the rod tip
        matters. Extends along +Z, matching this URDF's existing convention
@@ -377,7 +380,7 @@
   <link name="hydrophone_rod">
     <visual>
-      <origin rpy="0 0 0" xyz="0 0 0.05"/>
-      <geometry>
-        <cylinder radius="0.002" length="0.10"/>
+      <origin rpy="0 0 0" xyz="0 0 0.075"/>
+      <geometry>
+        <cylinder radius="0.002" length="0.15"/>
       </geometry>
       <material name="grey">
@@ -386,13 +389,14 @@
     </visual>
     <collision>
-      <origin rpy="0 0 0" xyz="0 0 0.05"/>
-      <geometry>
-        <cylinder radius="0.002" length="0.10"/>
+      <origin rpy="0 0 0" xyz="0 0 0.075"/>
+      <geometry>
+        <cylinder radius="0.002" length="0.15"/>
       </geometry>
     </collision>
   </link>
   <!-- Rod-tip reference frame (2026-08-24): a zero-size frame at the FAR
-       end of the rod (z=0.10 relative to virtual_endeffector, matching
-       the cylinder's own far face). MoveIt's planning group tip_link now
+       end of the rod (z=0.15 relative to virtual_endeffector as of the
+       2026-08-25 rod lengthening, matching the cylinder's own far face).
+       MoveIt's planning group tip_link now
        points HERE (see cyton_gamma_1500.srdf), not virtual_endeffector -
        reversing the original 2026-08-11 decision. IK/Cartesian targets
@@ -409,5 +413,5 @@
     <parent link="hydrophone_rod"/>
     <child link="hydrophone_tip"/>
-    <origin rpy="0 0 0" xyz="0 0 0.10"/>
+    <origin rpy="0 0 0" xyz="0 0 0.15"/>
   </joint>
   <link name="hydrophone_tip"/>

File: ros/src/cyton_description/urdf/cyton_gamma_1500_robot_sim7dof.xacro (robot description, xacro)
@@ -351,6 +351,9 @@
        rigidly to virtual_endeffector, representing the physical hydrophone
        probe used to measure ultrasound propagation at points on a skull
-       phantom. Dimensions are nominal design values (10cm length, 4mm
-       diameter), not independently calibrated - verify against the
+       phantom. Dimensions are nominal design values (15cm length, 4mm
+       diameter - lengthened from the original 10cm on 2026-08-25 to give
+       more standoff/collision clearance against the skull mesh, paired
+       with moving the skull's registration 10cm farther from base_link),
+       not independently calibrated - verify against the
        physical probe if precise real-world accuracy at the rod tip
        matters. Extends along +Z, matching this URDF's existing convention
@@ -365,7 +368,7 @@
   <link name="hydrophone_rod">
     <visual>
-      <origin rpy="0 0 0" xyz="0 0 0.05"/>
-      <geometry>
-        <cylinder radius="0.002" length="0.10"/>
+      <origin rpy="0 0 0" xyz="0 0 0.075"/>
+      <geometry>
+        <cylinder radius="0.002" length="0.15"/>
       </geometry>
       <material name="grey">
@@ -374,13 +377,14 @@
     </visual>
     <collision>
-      <origin rpy="0 0 0" xyz="0 0 0.05"/>
-      <geometry>
-        <cylinder radius="0.002" length="0.10"/>
+      <origin rpy="0 0 0" xyz="0 0 0.075"/>
+      <geometry>
+        <cylinder radius="0.002" length="0.15"/>
       </geometry>
     </collision>
   </link>
   <!-- Rod-tip reference frame (2026-08-24): a zero-size frame at the FAR
-       end of the rod (z=0.10 relative to virtual_endeffector, matching
-       the cylinder's own far face). MoveIt's planning group tip_link now
+       end of the rod (z=0.15 relative to virtual_endeffector as of the
+       2026-08-25 rod lengthening, matching the cylinder's own far face).
+       MoveIt's planning group tip_link now
        points HERE (see cyton_gamma_1500.srdf), not virtual_endeffector -
        reversing the original 2026-08-11 decision. IK/Cartesian targets
@@ -397,5 +401,5 @@
     <parent link="hydrophone_rod"/>
     <child link="hydrophone_tip"/>
-    <origin rpy="0 0 0" xyz="0 0 0.10"/>
+    <origin rpy="0 0 0" xyz="0 0 0.15"/>
   </joint>
   <link name="hydrophone_tip"/>

File: ros/src/cyton_description/urdf/cyton_gamma_1500_robot_uncalibrated.xacro (robot description, xacro)
@@ -377,6 +377,9 @@
        rigidly to virtual_endeffector, representing the physical hydrophone
        probe used to measure ultrasound propagation at points on a skull
-       phantom. Dimensions are nominal design values (10cm length, 4mm
-       diameter), not independently calibrated - verify against the
+       phantom. Dimensions are nominal design values (15cm length, 4mm
+       diameter - lengthened from the original 10cm on 2026-08-25 to give
+       more standoff/collision clearance against the skull mesh, paired
+       with moving the skull's registration 10cm farther from base_link),
+       not independently calibrated - verify against the
        physical probe if precise real-world accuracy at the rod tip
        matters. Extends along +Z, matching this URDF's existing convention
@@ -391,7 +394,7 @@
   <link name="hydrophone_rod">
     <visual>
-      <origin rpy="0 0 0" xyz="0 0 0.05"/>
-      <geometry>
-        <cylinder radius="0.002" length="0.10"/>
+      <origin rpy="0 0 0" xyz="0 0 0.075"/>
+      <geometry>
+        <cylinder radius="0.002" length="0.15"/>
       </geometry>
       <material name="grey">
@@ -400,13 +403,14 @@
     </visual>
     <collision>
-      <origin rpy="0 0 0" xyz="0 0 0.05"/>
-      <geometry>
-        <cylinder radius="0.002" length="0.10"/>
+      <origin rpy="0 0 0" xyz="0 0 0.075"/>
+      <geometry>
+        <cylinder radius="0.002" length="0.15"/>
       </geometry>
     </collision>
   </link>
   <!-- Rod-tip reference frame (2026-08-24): a zero-size frame at the FAR
-       end of the rod (z=0.10 relative to virtual_endeffector, matching
-       the cylinder's own far face). MoveIt's planning group tip_link now
+       end of the rod (z=0.15 relative to virtual_endeffector as of the
+       2026-08-25 rod lengthening, matching the cylinder's own far face).
+       MoveIt's planning group tip_link now
        points HERE (see cyton_gamma_1500.srdf), not virtual_endeffector -
        reversing the original 2026-08-11 decision. IK/Cartesian targets
@@ -416,5 +420,5 @@
     <parent link="hydrophone_rod"/>
     <child link="hydrophone_tip"/>
-    <origin rpy="0 0 0" xyz="0 0 0.10"/>
+    <origin rpy="0 0 0" xyz="0 0 0.15"/>
   </joint>
   <link name="hydrophone_tip"/>
